Commit message: switched to xacro files and removed redundant files

File: racecar_description/urdf/macros.xacro (robot description, xacro)
@@ -41,7 +41,5 @@
   <origin xyz="0 0 0" rpy="0 0 0" />
   <geometry>
-    <mesh>
-      <uri>package://racecar_description/meshes/chassis.STL</uri>
-    </mesh>
+    <mesh filename="$(find racecar_description)/meshes/chassis.STL" />
   </geometry>
 </xacro:macro>
@@ -49,7 +47,5 @@
   <origin xyz="0 0 0" rpy="0 0 0" />
   <geometry>
-    <mesh>
-      <uri>package://racecar_description/meshes/left_rear_wheel.STL</uri>
-    </mesh>
+    <mesh filename="$(find racecar_description)/meshes/left_rear_wheel.STL" />
   </geometry>
 </xacro:macro>
@@ -57,7 +53,5 @@
   <origin xyz="0 0 0" rpy="0 0 0" />
   <geometry>
-    <mesh>
-      <uri>package://racecar_description/meshes/right_rear_wheel.STL</uri>
-    </mesh>
+    <mesh filename="$(find racecar_description)/meshes/right_rear_wheel.STL" />
   </geometry>
 </xacro:macro>
@@ -65,7 +59,5 @@
   <origin xyz="0 0 0" rpy="0 0 0" />
   <geometry>
-    <mesh>
-      <uri>package://racecar_description/meshes/left_front_wheel.STL</uri>
-    </mesh>
+    <mesh filename="$(find racecar_description)/meshes/left_front_wheel.STL" />
   </geometry>
 </xacro:macro>
@@ -73,7 +65,5 @@
   <origin xyz="0 0 0" rpy="0 0 0" />
   <geometry>
-    <mesh>
-      <uri>package://racecar_description/meshes/right_front_wheel.STL</uri>
-    </mesh>
+    <mesh filename="$(find racecar_description)/meshes/right_front_wheel.STL" />
   </geometry>
 </xacro:macro>
@@ -81,7 +71,5 @@
   <origin xyz="0 0 0" rpy="0 0 0" />
   <geometry>
-    <mesh>
-      <uri>package://racecar_description/meshes/left_steering_hinge.STL</uri>
-    </mesh>
+    <mesh filename="$(find racecar_description)/meshes/left_steering_hinge.STL" />
   </geometry>
 </xacro:macro>
@@ -89,7 +77,5 @@
   <origin xyz="0 0 0" rpy="0 0 0" />
   <geometry>
-    <mesh>
-      <uri>package://racecar_description/meshes/right_steering_hinge.STL</uri>
-    </mesh>
+    <mesh filename="$(find racecar_description)/meshes/right_steering_hinge.STL" />
   </geometry>
 </xacro:macro>

File: racecar_description/urdf/racecar.xacro (robot description, xacro)
@@ -1,5 +1,5 @@
 <?xml version="1.0"?>
 <robot name="racecar" xmlns:xacro="http://www.ros.org/wiki/xacro">
-  <xacro:include filename="$(find racecar_description)/urdf/macros.xacro.xml" />
+  <xacro:include filename="$(find racecar_description)/urdf/macros.xacro" />
   <!-- Add chassis and it's inertia link -->
   <link name="base_link" />
@@ -34,5 +34,5 @@
       <material name="black" />
     </visual>
-    <collision>
+    <collision>robot
       <xacro:left_wheels_collision_geometry />
     </collision>
@@ -159,7 +159,5 @@
       <origin xyz="0 0 0" rpy="0 0 0"/>
       <geometry>
-        <mesh>
-          <uri>package://racecar_description/meshes/hokuyo.dae</uri>
-        </mesh>
+        <mesh filename="package://racecar_description/meshes/hokuyo.dae"/>
         <material name="grey" />
       </geometry>
@@ -230,4 +228,52 @@
   <!-- Add the remaining xacros -->
   <xacro:include filename="$(find racecar_description)/urdf/racecar.gazebo" />
-  <xacro:include filename="$(find racecar_description)/urdf/materials.xacro.xml" />
+  <xacro:include filename="$(find racecar_description)/urdf/materials.xacro" />
+  <!-- Add ros2 xacros -->
+  <ros2_control name="GazeboSystem" type="system">
+    <hardware>
+      <plugin>gazebo_ros2_control/GazeboSystem</plugin>
+    </hardware>
+    <joint name="left_rear_wheel_joint">
+      <command_interface name="effort">
+        <param name="min">-1000</param>
+        <param name="max">1000</param>
+      </command_interface>
+      <state_interface name="velocity"/>
+    </joint>
+    <joint name="right_rear_wheel_joint">
+      <command_interface name="effort">
+        <param name="min">-1000</param>
+        <param name="max">1000</param>
+      </command_interface>
+      <state_interface name="velocity"/>
+    </joint>
+    <joint name="left_front_wheel_joint">
+      <command_interface name="effort">
+        <param name="min">-1000</param>
+        <param name="max">1000</param>
+      </command_interface>
+      <state_interface name="velocity"/>
+    </joint>
+    <joint name="right_front_wheel_joint">
+      <command_interface name="effort">
+        <param name="min">-1000</param>
+        <param name="max">1000</param>
+      </command_interface>
+      <state_interface name="velocity"/>
+    </joint>
+    <joint name="right_steering_hinge_joint">
+      <command_interface name="effort">
+        <param name="min">-1000</param>
+        <param name="max">1000</param>
+      </command_interface>
+      <state_interface name="position"/>
+    </joint>
+    <joint name="left_steering_hinge_joint">
+      <command_interface name="effort">
+        <param name="min">-1000</param>
+        <param name="max">1000</param>
+      </command_interface>
+      <state_interface name="position"/>
+    </joint>
+  </ros2_control>
 </robot>
