Commit message: correct xacro

File: racecar_description/urdf/racecar.xacro (robot description, xacro)
@@ -34,5 +34,5 @@
       <material name="black" />
     </visual>
-    <collision>robot
+    <collision>
       <xacro:left_wheels_collision_geometry />
     </collision>

Commit message: udpate joint limits

File: racecar_description/urdf/racecar.xacro (robot description, xacro)
@@ -82,5 +82,5 @@
     <child link="left_steering_hinge" />
     <axis xyz="-1 0 0" />
-    <limit lower="-1.0" upper="1.0" effort="10" velocity="100" />
+    <limit lower="-0.4" upper="0.4" effort="10" velocity="100" />
   </joint>
   <xacro:steering_hinge_transmission name="left_steering_hinge" />
@@ -100,5 +100,5 @@
     <child link="right_steering_hinge" />
     <axis xyz="-1 0 0" />
-    <limit lower="-1.0" upper="1.0" effort="10" velocity="100" />
+    <limit lower="-0.4" upper="0.4" effort="10" velocity="100" />
   </joint>
   <xacro:steering_hinge_transmission name="right_steering_hinge" />

Commit message: Added additional config files

File: racecar_description/urdf/racecar.xacro (robot description, xacro)
@@ -171,5 +171,5 @@
   </joint>
   <!-- zed camera -->
-  <link name="zed_camera_link">
+  <link name="camera_link">
     <inertial>
       <mass value="1e-5" />
@@ -191,15 +191,16 @@
     </visual>
   </link>
-  <joint name="zed_camera_joint" type="fixed">
+  <joint name="camera_joint" type="fixed">
     <origin xyz="0.390 0 0.04" rpy="0 0 0"/>
     <parent link="chassis"/>
-    <child link="zed_camera_link"/>
-    <axis xyz="0 0 1" />
-    <!-- <limit lower="0.0" upper="0.0" effort="0.0" velocity="0.0" /> -->
+    <child link="camera_link"/>
+    <axis xyz="0 0 1" />
+     <limit lower="0.0" upper="0.0" effort="0.0" velocity="0.0" />
   </joint>
   <!-- zed camera lenses -->
   <!-- It seems these have to have a non-zero mass to have a camera attached? -->
-  <link name="camera_link"><!-- this needs to match the name in zed_wrapper/zed_tf.launch -->
-    <inertial>
+  <!--
+  <link name="camera_link">
+	  <inertial>
       <mass value="1e-5" />
       <origin xyz="0 0 0" rpy="0 0 0"/>
@@ -226,4 +227,5 @@
     <axis xyz="0 0 1" />
   </joint>
+	  -->
   <!-- Add the remaining xacros -->
   <xacro:include filename="$(find racecar_description)/urdf/racecar.gazebo" />

Commit message: Renamed depth image node to avoid confusion (node was previously named scan)

File: racecar_description/urdf/racecar.xacro (robot description, xacro)
@@ -145,29 +145,4 @@
   </joint>
   <!-- <xacro:wheel_transmission name="right_front_wheel" /> -->
-  <!-- Add Hokuyo laser scanner -->
-  <link name="laser">
-    <inertial>
-      <xacro:hokuyo_inertial_params />
-    </inertial>
-    <collision>
-      <origin xyz="0 0 0" rpy="0 0 0"/>
-      <geometry>
-        <box size="0.1 0.1 0.1"/>
-      </geometry>
-    </collision>
-    <visual>
-      <origin xyz="0 0 0" rpy="0 0 0"/>
-      <geometry>
-        <mesh filename="package://racecar_description/meshes/hokuyo.dae"/>
-        <material name="grey" />
-      </geometry>
-    </visual>
-  </link>
-  <joint name="hokuyo_joint" type="fixed">
-    <origin xyz="0.265 0.0 0.075" rpy="0 0 0"/>
-    <parent link="chassis" />
-    <child link="laser" />
-    <axis xyz="0 0 1" />
-  </joint>
   <!-- zed camera -->
   <link name="camera_link">

Commit message: Removed camera and depthimage from launch file

File: racecar_description/urdf/racecar.xacro (robot description, xacro)
@@ -167,5 +167,5 @@
   </link>
   <joint name="camera_joint" type="fixed">
-    <origin xyz="0.390 0 0.04" rpy="0 0 0"/>
+    <origin xyz="0.3429 0 0.1524" rpy="0 0 0"/>
     <parent link="chassis"/>
     <child link="camera_link"/>
